Commit message: Update ur5e_robotiq.urdf.xacro
Fix 90 deg offset to match reality and bullet simulation

File: urdf/ur5e_robotiq.urdf.xacro (robot description, xacro)
@@ -10,5 +10,5 @@
     <parent link="tool0" />
     <child link="robotiq_arg2f_base_link" />
-    <origin xyz="0 0 0" rpy="0 0 0" />
+    <origin xyz="0 0 0" rpy="0 1.57079632679 0" />
   </joint>
   <!-- Make gripper controllable in Gazebo -->

Commit message: Only publish relevant joint states. Fix ee pose again.

File: urdf/ur5e_robotiq.urdf.xacro (robot description, xacro)
@@ -10,5 +10,5 @@
     <parent link="tool0" />
     <child link="robotiq_arg2f_base_link" />
-    <origin xyz="0 0 0" rpy="0 1.57079632679 0" />
+    <origin xyz="0 0 0" rpy="0 0 1.57079632679" />
   </joint>
   <!-- Make gripper controllable in Gazebo -->
